File: jarduino2/jard_485_slave/board/jard_rs485_slave_mods/jard_rs485_slave_mods.sch (KiCad schematic (older format))
At the start: 20 parts, among them J1 NETWORK IN, J2 NETWORK OUT, J4 LED, J5 Niveau bas, J6 Electrovanne 12V, J7 Niveau Haut, Q1 TIP41C, U1 BPC_Mod485

Commit message: ?
Connections:
- net GND: now also J1.4 (Pin_4), J2.4 (Pin_4)
Changed lines of the file:
@@
 	1900 1700 1900 2600
 Wire Wire Line
-	1900 2600 1200 2600
+	1900 2600 1800 2600
 Wire Wire Line
 	1800 2500 1800 1500
@@
 Wire Wire Line
 	4400 3900 4400 3950
+$Comp
+L power:GND #PWR?
+U 1 1 63E899D1
+P 1800 2800
+F 0 "#PWR?" H 1800 2550 50  0001 C CNN
+F 1 "GND" H 1805 2627 50  0000 C CNN
+F 2 "" H 1800 2800 50  0001 C CNN
+F 3 "" H 1800 2800 50  0001 C CNN
+	1    1800 2800
+	1    0    0    -1
+$EndComp
+Connection ~ 1800 2600
+Wire Wire Line
+	1800 2600 1200 2600
+Wire Wire Line
+	1800 2600 1800 2800
 $EndSCHEMATC

Commit message: Redesign avec 1 MOS et 2 entrées flowmeter Dimensions ajustées suite proto mécanique Ajout datasheets
Parts:
- removed C11: 10nF, Capacitor_THT:C_Disc_D5.0mm_W2.5mm_P2.50mm, symbol Device:C
- removed C12: 20µF, Capacitor_THT:CP_Radial_D12.5mm_P5.00mm, symbol Device:CP
- removed J7: Niveau Haut, TerminalBlock_Phoenix:TerminalBlock_Phoenix_MKDS-3-2-5.08_1x02_P5.08mm_Horizontal, symbol Connector:Screw_Terminal_01x02
- removed Q1: TIP41C, Package_TO_SOT_THT:TO-220-3_Vertical, symbol Transistor_BJT:TIP41C
- removed R3: 50, Resistor_THT:R_Axial_DIN0309_L9.0mm_D3.2mm_P2.54mm_Vertical, symbol Device:R
- added D2: D, Diode_THT:D_A-405_P2.54mm_Vertical_AnodeUp, symbol Device:D
- added J4: LED, Connector_PinHeader_2.54mm:PinHeader_1x02_P2.54mm_Vertical, symbol Connector_Generic:Conn_01x02
- added J5: Debit, TerminalBlock_Phoenix:TerminalBlock_Phoenix_MPT-0,5-3-2.54_1x03_P2.54mm_Horizontal, symbol Connector_Generic:Conn_01x03
- added Q1: BPC_2N2222A, Package_TO_SOT_THT:TO-18-3, symbol bpc:BPC_2N2222A
- added Q2: P03P4L-04, Package_TO_SOT_THT:TO-220-3_Vertical, symbol bpc:P03P4L-04
- added R2: 150, Resistor_THT:R_Axial_DIN0309_L9.0mm_D3.2mm_P2.54mm_Vertical, symbol Device:R
- added R5: 100, Resistor_THT:R_Axial_DIN0309_L9.0mm_D3.2mm_P2.54mm_Vertical, symbol Device:R
- added R8, R9: 100k, Resistor_THT:R_Axial_DIN0309_L9.0mm_D3.2mm_P2.54mm_Vertical, symbol Device:R
- added U2: BPC_DHT22, bpc:BPC_DHT22, symbol bpc:BPC_DHT22
- J1, J2: footprint TerminalBlock_Phoenix:TerminalBlock_Phoenix_MKDS-3-4-5.08_1x04_P5.08mm_Horizontal -> TerminalBlock_Phoenix:TerminalBlock_Phoenix_MPT-0,5-4-2.54_1x04_P2.54mm_Horizontal
- J6: renamed from J5; value Niveau bas -> Niveau; footprint TerminalBlock_Phoenix:TerminalBlock_Phoenix_MKDS-3-2-5.08_1x02_P5.08mm_Horizontal -> TerminalBlock_Phoenix:TerminalBlock_Phoenix_MPT-0,5-3-2.54_1x03_P2.54mm_Horizontal; symbol Connector:Screw_Terminal_01x02 -> Connector_Generic:Conn_01x03
- J7: renamed from J6; footprint TerminalBlock_Phoenix:TerminalBlock_Phoenix_MKDS-3-2-5.08_1x02_P5.08mm_Horizontal -> TerminalBlock_Phoenix:TerminalBlock_Phoenix_MPT-0,5-2-2.54_1x02_P2.54mm_Horizontal
- renumbered C5 to C1, C7 to C2, J4 to J3, R2 to R1, R1 to R3, R5 to R7
Connections:
- net CMD_EV: now also A1.10 (D7), R5.2; no longer A1.7 (D4)
- net GND: now also J3.2 (Pin_2), J6.3 (Pin_3), J7.1 (Pin_1), R6.2, D2.2 (A), J4.2 (Pin_2), J5.3 (Pin_3), Q1.1, U2.4 (GND); no longer J3.1 (Pin_1), J6.1 (Pin_1), R4.2
- net IN_LVL_HIGH: now also A1.6 (D3), J6.2 (Pin_2), R8.2; no longer A1.9 (D6), R6.2
- net IN_LVL_LOW: now also A1.5 (D2), J6.1 (Pin_1); no longer A1.10 (D7), J6.2 (Pin_2)
- net TXEN: now also A1.9 (D6); no longer A1.5 (D2)
- net Vcc: now also R4.1, J5.1 (Pin_1), R8.1, U2.1 (VDD); no longer R6.1
- net at A1.30 (VIN), C1.2, C2.1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: now also Q2.3 (S), R9.1; no longer J7.2 (Pin_2)
- net LED1: now reaches R1.1
- net LED1: now also A1.11 (D8); no longer J3.2 (Pin_2)
- net at R1.2: now also J3.1 (Pin_1); no longer A1.8 (D5)
- net LED2: now reaches A1.12 (D9)
- net LED2: now also R2.1
- net TEMP: now reaches A1.13 (D10)
- net TEMP: now also U2.2 (DATA)
- new net: D2.1 (K), J7.2 (Pin_2), Q2.2 (D)
- new net: Q1.3, Q2.1 (G), R9.2
- new net: Q1.2, R5.1, R6.1
- new net: J4.1 (Pin_1), R2.2
- new net FLOW_IN: A1.7 (D4), J5.2 (Pin_2), R4.2
- no-connect marks 0 -> 16
Other:
- moved on the sheet: J3, J7, R1, R7
