File: jarduino2/jard_485_slave/board/jard_rs485_slave_at328/ES.kicad_sch (KiCad schematic)
At the start: 21 parts

Commit message: Changement empreinte de D2 (trous + gros et 12mm long) Dessin sérigraphie J2 (sens de la sonde)
Parts:
- C?: RefFabricant C0603X102J5GACAUTO -> C0603C104K1RACTU; RefFournisseur 2219417 -> 4199453
Changed lines of the file:
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@@
       (effects (font (size 1.27 1.27)) hide)
     )
-    (property "RefFabricant" "C0603X102J5GACAUTO" (at 204.47 105.41 0)
+    (property "RefFabricant" "C0603C104K1RACTU" (at 204.47 105.41 0)
       (effects (font (size 1.27 1.27)) hide)
     )
-    (property "RefFournisseur" "2219417" (at 204.47 105.41 0)
+    (property "RefFournisseur" "4199453" (at 204.47 105.41 0)
       (effects (font (size 1.27 1.27)) hide)
     )
