File: jarduino2/jard_485_slave/board/jard_rs485_slave_mods2/uc.kicad_sch (KiCad schematic)
At the start: 14 parts, among them J1 POWER

Commit message: Modification titre du schéma + Nomenclature
Parts:
- J1: Fabricant (none) -> PHOENIX CONTACT; Fournisseur (none) -> Farnell
Changed lines of the file:
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@@
+      (effects (font (size 1.27 1.27)) hide)
+    )
+    (property "Description" "Bornier 2 contacts 5.08mm" (at 33.02 39.37 0)
+      (effects (font (size 1.27 1.27)) hide)
+    )
+    (property "Fabricant" "PHOENIX CONTACT" (at 33.02 39.37 0)
+      (effects (font (size 1.27 1.27)) hide)
+    )
+    (property "Fournisseur" "Farnell" (at 33.02 39.37 0)
       (effects (font (size 1.27 1.27)) hide)
     )
