File: jarduino2/jard_wemos/board/jard_wemos.kicad_sch (KiCad schematic)
At the start: 30 parts, among them J1 Conn_01x05, J2 LEDs, Q1 BPC_IPP034N03L, U1 BPC_Alim3_3V, U2 WeMos_D1_mini, U3 24LC01

Commit message: Note à faire
Other:
- note added: "A faire: Relier D0 et RST (réveil de veille) Passer en CMS"
Changed lines of the file:
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@@
     (stroke (width 0) (type default))
+  )
+  (text "A faire:\n\nRelier D0 et RST (réveil de veille)\nPasser en CMS"
+    (at 30.48 181.61 0)
+    (effects (font (size 1.27 1.27)) (justify left bottom))
   )
   (global_label "LED_ROUGE" (shape output) (at 143.51 139.7 0)
