File: lcduino/hard/lcduino.kicad_pcb (KiCad board)
At the start: 2 copper layers, 86 x 50 mm, 31 parts, among them J1 Alim 12V, J2 ILI9341, J3 SD, J4 SD, Q1 BPC_FMMT38C, Q2 AO3401A, U1 NodeMCUs, U2 BPC_Alim3_3V

Commit message: Changement connecteur header en socket
Parts:
- J2: footprint Connector_PinHeader_2.54mm:PinHeader_1x14_P2.54mm_Vertical -> Connector_PinSocket_2.54mm:PinSocket_1x14_P2.54mm_Vertical
- J3: footprint Connector_PinHeader_2.54mm:PinHeader_1x04_P2.54mm_Vertical -> Connector_PinSocket_2.54mm:PinSocket_1x04_P2.54mm_Vertical
- moved J4 60.8 mm to (193.5, 105.0), turned to 180 degrees
- moved R6 52.0 mm to (191.5, 98.0), turned to -90 degrees
- moved D3 51.9 mm to (191.4, 97.9), turned to -90 degrees
- moved C5 20.0 mm to (176.0, 96.0)
- moved U1 20.0 mm to (159.2, 87.6)
- moved C7 19.8 mm to (175.2, 103.0)
- moved C6 19.8 mm to (175.2, 102.0)

Commit message: Fin placement et routage complet A valider
Parts:
- C2, C3: moved to F.Cu
- D1: moved to B.Cu
- moved D1 15.2 mm to (139.7, 103.9)
- moved C10 8.49 mm to (206.4, 83.1)
- moved J4 8.30 mm to (197.9, 98.0), turned to -90 degrees
- moved C1 8.07 mm to (156.1, 112.5)
- moved C13 7.15 mm to (208.8, 100.3), turned to -90 degrees
- moved C2 5.26 mm to (150.3, 112.2)
- moved C11 5.01 mm to (193.4, 80.7)
- moved Q2 5.01 mm to (198.1, 80.7)
- moved R3 5.01 mm to (198.0, 75.7)
- moved R4 5.01 mm to (198.0, 77.7)
- moved J1 4.24 mm to (137.0, 108.0), turned to 0 degrees
- moved R2 4.08 mm to (199.0, 84.4), turned to 90 degrees
- moved D2 3.73 mm to (145.1, 116.9)
- moved C9 3.28 mm to (208.8, 82.6)
- moved J2 3.11 mm to (212.0, 81.5)
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Routing:
- net LCD_MISO: track 0.00 -> 121.3 mm, vias 0 -> 2
- net LCD_SCK: track 0.00 -> 116.9 mm, vias 0 -> 1
- net +3.3V: track 0.00 -> 114.4 mm, vias 0 -> 2
- net LCD_MOSI: track 0.00 -> 107.5 mm, vias 0 -> 1
- net LCD_CS: track 0.00 -> 76.9 mm
- net LCD_DC: track 0.00 -> 75.8 mm
- net BUTTON: track 0.00 -> 68.8 mm, vias 0 -> 1
- net BUZZER: track 0.00 -> 57.7 mm, vias 0 -> 4
- net CMD_PWR_LCD: track 0.00 -> 47.0 mm
- net LCD_VCC: track 0.00 -> 40.7 mm, vias 0 -> 2
- net SD_CS: track 0.00 -> 25.7 mm
- net Net-(D1-A2): track 0.00 -> 17.4 mm
- net Net-(D2-K): track 0.00 -> 15.7 mm
- net Net-(J2-Pin_4): track 0.00 -> 15.6 mm, vias 0 -> 1
- net GND: track 0.00 -> 14.5 mm, vias 0 -> 3
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- added copper zone on B.Cu, net GND
- added copper zone on F.Cu, net GND
Other:
- outline, holes or cut-outs redrawn
- board text added: "+5-12V"
- board text added: "Button"
- board text added: "Gnd"
- board text added: "POWER"

Commit message: Finalisation et revue
Routing:
- net BUTTON: track 68.8 -> 72.7 mm
- net GND: track 14.5 -> 17.8 mm, vias 3 -> 82
- net LCD_SCK: track 116.9 -> 115.8 mm
- net LCD_MISO: track 121.3 -> 120.6 mm
